File: SensoriFeatherWing.kicad_pcb (KiCad board)
At the start: 2 copper layers, 50.8 x 22.9 mm, 20 parts, among them J2 Conn_01x04, J3 Conn_01x04, J4 Conn_01x04, J5 5-12 V, max. 5A, J6 Screw_Terminal_01x02, J7 Conn_01x02_Male, SW1 B3U-1000P, SW2 SW_SPST, U1 LTC2850xMS8, U2 MIC5219-5.0YM5

Commit message: updated silkscreen
Parts:
- moved G*** 1.82 mm to (513.3, 343.8)
Other:
- board text added: "3V3"
- board text added: "RST"
- board text added: "VUSB"
Changed lines of the file:
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@@
   (general
     (thickness 1.6)
-    (drawings 50)
+    (drawings 68)
     (tracks 86)
     (zones 0)
@@
   )
   (setup
-    (last_trace_width 0.4572)
+    (last_trace_width 0.25)
     (user_trace_width 0.254)
     (user_trace_width 0.3048)
@@
       (effects (font (size 1 1) (thickness 0.15)))
     )
-    (fp_text user %R (at 0 0 90) (layer F.Fab)
-      (effects (font (size 0.5 0.5) (thickness 0.08)))
-    )
     (fp_line (start -1.9 -0.85) (end -1.9 0.85) (layer F.SilkS) (width 0.12))
     (fp_line (start 0.2 0) (end 0.45 0) (layer F.Fab) (width 0.1))
@@
     (fp_line (start -1.9 0.85) (end 1.25 0.85) (layer F.SilkS) (width 0.12))
     (fp_line (start -1.9 -0.85) (end 1.25 -0.85) (layer F.SilkS) (width 0.12))
+    (fp_text user %R (at 0 0 90) (layer F.Fab)
+      (effects (font (size 0.5 0.5) (thickness 0.08)))
+    )
     (pad 2 smd rect (at 1.25 0 270) (size 1 1) (layers F.Cu F.Paste F.Mask)
       (net 32 "Net-(C3-Pad1)"))
@@
   )
   (module Gretchen:gretchen_logo_bmp (layer B.Cu)
-    (at 511.556 344.17 180)
+    (at 513.334 343.789 180)
     (fp_text reference G*** (at 0 0) (layer B.SilkS) hide
       (effects (font (size 1.524 1.524) (thickness 0.3)) (justify mirror))
@@
       (xy -4.180627 1.4431) (xy -3.980001 1.459616) (xy -3.803067 1.437107)) (layer B.SilkS) (width 0.01))
   )
-  (module Module:Adafruit_Feather_WithMountingHoles locked (layer F.Cu)
+  (module Module:Adafruit_Feather_WithMountingHoles (layer F.Cu)
     (at 495.3 351.79 90)
     (descr "Common footprint for the Adafruit Feather series of boards, https://learn.adafruit.com/adafruit-feather/feather-specification")
@@
     )
   )
+  (gr_circle (center 510.54 331.47) (end 511.632495 331.47) (layer F.SilkS) (width 0.18))
+  (gr_line (start 499.872 349.758) (end 498.729 350.901) (layer B.SilkS) (width 0.18))
+  (gr_line (start 500.507 349.758) (end 499.872 349.758) (layer B.SilkS) (width 0.18))
+  (gr_line (start 497.332 349.758) (end 498.983 349.758) (layer B.SilkS) (width 0.18))
+  (gr_line (start 496.443 350.647) (end 497.332 349.758) (layer B.SilkS) (width 0.18))
+  (gr_text RST (at 498.983 349.504 270) (layer B.SilkS)
+    (effects (font (size 0.8 0.8) (thickness 0.18)) (justify left mirror))
+  )
+  (gr_text 3V3 (at 500.507 349.504 270) (layer B.SilkS)
+    (effects (font (size 0.8 0.8) (thickness 0.18)) (justify left mirror))
+  )
+  (gr_line (start 524.637 332.613) (end 525.018 332.232) (layer B.SilkS) (width 0.18))
+  (gr_line (start 524.637 332.994) (end 524.637 332.613) (layer B.SilkS) (width 0.18))
+  (gr_line (start 529.463 332.613) (end 529.082 332.232) (layer B.SilkS) (width 0.18))
+  (gr_line (start 529.463 332.994) (end 529.463 332.613) (layer B.SilkS) (width 0.18))
+  (gr_text GND (at 502.92 350.52 270) (layer B.SilkS)
+    (effects (font (size 0.8 0.8) (thickness 0.18)) (justify left mirror))
+  )
+  (gr_text DI (at 530.86 350.52 270) (layer B.SilkS)
+    (effects (font (size 0.8 0.8) (thickness 0.18)) (justify left mirror))
+  )
+  (gr_text RO (at 528.32 350.52 270) (layer B.SilkS)
+    (effects (font (size 0.8 0.8) (thickness 0.18)) (justify left mirror))
+  )
+  (gr_text RST (at 495.3 350.139) (layer F.SilkS)
+    (effects (font (size 0.8 0.8) (thickness 0.18)))
+  )
+  (gr_text VUSB (at 510.54 332.74 270) (layer B.SilkS)
+    (effects (font (size 0.8 0.8) (thickness 0.18)) (justify right mirror))
+  )
+  (gr_text GND (at 502.92 350.139) (layer F.SilkS)
+    (effects (font (size 0.8 0.8) (thickness 0.18)))
+  )
+  (gr_text 3V3 (at 497.84 350.139) (layer F.SilkS)
+    (effects (font (size 0.8 0.8) (thickness 0.18)))
+  )
   (gr_poly (pts (xy 506.9332 341.8332) (xy 506.4252 341.8332) (xy 506.6792 341.5792)) (layer F.SilkS) (width 0.18))
-  (gr_line (start 518.414 347.472) (end 517.398 349.25) (layer B.SilkS) (width 0.18))
-  (gr_line (start 519.43 349.25) (end 518.414 347.472) (layer B.SilkS) (width 0.18))
-  (gr_line (start 517.398 349.25) (end 519.43 349.25) (layer B.SilkS) (width 0.18))
-  (gr_text ! (at 518.414 348.615) (layer B.SilkS)
+  (gr_line (start 519.938 346.964) (end 518.922 348.742) (layer B.SilkS) (width 0.18))
+  (gr_line (start 520.954 348.742) (end 519.938 346.964) (layer B.SilkS) (width 0.18))
+  (gr_line (start 518.922 348.742) (end 520.954 348.742) (layer B.SilkS) (width 0.18))
+  (gr_text ! (at 519.938 348.107) (layer B.SilkS)
     (effects (font (size 0.8 0.8) (thickness 0.18)) (justify mirror))
   )
-  (gr_text "Don’t connect to USB\nand back-power the Feather\nat the same time" (at 516.763 348.361) (layer B.SilkS)
+  (gr_text "Don’t connect to USB and\nback-power the Feather\nat the same time" (at 518.668 347.726) (layer B.SilkS)
     (effects (font (size 0.8 0.8) (thickness 0.18)) (justify left mirror))
   )
@@
     (effects (font (size 0.8 0.8) (thickness 0.18)))
   )
-  (gr_text RESET (at 504.19 349.885) (layer F.SilkS)
+  (gr_text RESET (at 501.142 347.726 90) (layer F.SilkS)
     (effects (font (size 0.8 0.8) (thickness 0.18)))
   )
-  (gr_text DE (at 524.764 334.01) (layer B.SilkS)
+  (gr_text DE (at 524.764 334.01 270) (layer B.SilkS)
     (effects (font (size 0.8 0.8) (thickness 0.18)) (justify mirror))
   )
-  (gr_text ~RE (at 529.717 334.01) (layer B.SilkS)
+  (gr_text ~RE (at 529.463 334.01 270) (layer B.SilkS)
     (effects (font (size 0.8 0.8) (thickness 0.18)) (justify mirror))
   )
@@
     (effects (font (size 0.8 0.8) (thickness 0.18)) (justify right))
   )
-  (gr_text "Nov 2020, rev B" (at 516.89 341.376) (layer B.SilkS)
+  (gr_text "Nov 2020, rev B" (at 518.668 341.376) (layer B.SilkS)
     (effects (font (size 0.8 0.8) (thickness 0.18)) (justify left mirror))
   )
-  (gr_text DI (at 530.86 349.885) (layer F.SilkS)
+  (gr_text DI (at 530.86 350.139) (layer F.SilkS)
     (effects (font (size 0.8 0.8) (thickness 0.18)))
   )
-  (gr_text RO (at 528.32 349.885) (layer F.SilkS)
+  (gr_text RO (at 528.32 350.139) (layer F.SilkS)
     (effects (font (size 0.8 0.8) (thickness 0.18)))
   )
@@
     (effects (font (size 0.8 0.8) (thickness 0.18)))
   )
-  (gr_text "Sensorimotor FeatherWing" (at 517.017 339.598) (layer B.SilkS)
+  (gr_text "Sensorimotor FeatherWing" (at 518.668 339.598) (layer B.SilkS)
     (effects (font (size 1.2 1.2) (thickness 0.22)) (justify left mirror))
   )

Commit message: Update
Parts:
- added R3: 120 Ω, Resistor_SMD:R_0805_2012Metric_Pad1.20x1.40mm_HandSolder, F.Cu at (537.2, 341.6)
Routing:
- net VBUS: track 60.5 -> 75.0 mm, vias 0 -> 1
- net /B: track 27.1 -> 28.6 mm
- net /A: track 29.5 -> 29.0 mm
