File: SensoriFeatherWing.sch (KiCad schematic (older format))
At the start: 18 parts, among them J2 Conn_01x04, J3 Conn_01x04, J4 Conn_01x04, J5 5-12 V, max. 5A, J6 Screw_Terminal_01x02, J7 Conn_01x02_Male, SW1 B3U-1000P, SW2 SW_SPST, U1 LTC2850xMS8, U2 MIC5219-5.0YM5

Commit message: Update
Parts:
- added R3: 120 Ω, Resistor_SMD:R_0805_2012Metric_Pad1.20x1.40mm_HandSolder, symbol Device:R
- C1: DKPN (none) -> 311-4266-1-ND
- C2: DKPN (none) -> 311-3497-1-ND
- C3: DKPN (none) -> 1276-2872-1-ND
- J2, J3, J4: DKPN (none) -> WM18888-ND
- SW2: DKPN (none) -> 2223-DS04-254-1L-01BK-ND
- U1: DKPN (none) -> LTC2850IMS8#PBF-ND
Connections:
- net A: now also R3.2
- net B: now also R3.1
Other:
- note added: "End Termination Resistor (optional)\n~~ 120 Ohm\nPTH and SMD option"
- note removed: "End Termination Resistor (optional)\n~ 120 Ohm"
- note removed: "TODO:\n- Read datasheet of LDO -> caps? ESR?"
Changed lines of the file:
@@
 encoding utf-8
 Sheet 1 1
-Title "LTC2850 Breakout"
+Title "Sensori FeatherWing"
 Date "2020-11-14"
 Rev "B"
 Comp ""
-Comment1 ""
+Comment1 "Author: Emil Bergold"
 Comment2 ""
 Comment3 ""
@@
 F 2 "Package_SO:MSOP-8_3x3mm_P0.65mm" H 4450 1300 50  0001 C CNN
 F 3 "https://www.analog.com/media/en/technical-documentation/data-sheets/285012fe.pdf" H 3950 2300 50  0001 C CNN
+F 4 "LTC2850IMS8#PBF-ND" H 4450 2200 50  0001 C CNN "DKPN"
 	1    4450 2200
 	1    0    0    -1
@@
 F 2 "Connector_Molex:Molex_SPOX_5267-04A_1x04_P2.50mm_Vertical" H 6300 1850 50  0001 C CNN
 F 3 "~" H 6300 1850 50  0001 C CNN
+F 4 "WM18888-ND" H 6300 1850 50  0001 C CNN "DKPN"
 	1    6300 1850
 	1    0    0    -1
@@
 F 2 "Connector_Molex:Molex_SPOX_5267-04A_1x04_P2.50mm_Vertical" H 6300 2300 50  0001 C CNN
 F 3 "~" H 6300 2300 50  0001 C CNN
+F 4 "WM18888-ND" H 6300 2300 50  0001 C CNN "DKPN"
 	1    6300 2300
 	1    0    0    -1
@@
 F 2 "Connector_Molex:Molex_SPOX_5267-04A_1x04_P2.50mm_Vertical" H 6300 2750 50  0001 C CNN
 F 3 "~" H 6300 2750 50  0001 C CNN
+F 4 "WM18888-ND" H 6300 2750 50  0001 C CNN "DKPN"
 	1    6300 2750
 	1    0    0    -1
@@
 F 2 "Capacitor_SMD:C_0805_2012Metric_Pad1.18x1.45mm_HandSolder" H 4800 1450 50  0001 C CNN
 F 3 "~" H 4800 1450 50  0001 C CNN
+F 4 "311-4266-1-ND" H 4800 1450 50  0001 C CNN "DKPN"
 	1    4800 1450
 	0    1    1    0
@@
 A
 Wire Wire Line
-	4900 3750 5200 3750
-Wire Wire Line
-	5500 3750 5800 3750
+	4900 3750 5100 3750
+Wire Wire Line
+	5500 3750 5600 3750
 Text Label 5800 3750 0    50   ~ 0
 B
-Text Notes 5250 4050 0    50   ~ 0
-End Termination Resistor (optional)\n~ 120 Ohm
+Text Notes 5200 4450 0    50   ~ 0
+End Termination Resistor (optional)\n~~ 120 Ohm\nPTH and SMD option
 Wire Wire Line
 	7750 1550 8300 1550
@@
 F 2 "Capacitor_SMD:C_0805_2012Metric_Pad1.18x1.45mm_HandSolder" H 7400 4600 50  0001 C CNN
 F 3 "~" H 7400 4600 50  0001 C CNN
+F 4 "311-3497-1-ND" H 7400 4600 50  0001 C CNN "DKPN"
 	1    7400 4600
 	1    0    0    -1
@@
 F 2 "Capacitor_SMD:C_0805_2012Metric_Pad1.18x1.45mm_HandSolder" H 9200 4600 50  0001 C CNN
 F 3 "~" H 9200 4600 50  0001 C CNN
+F 4 "1276-2872-1-ND" H 9200 4600 50  0001 C CNN "DKPN"
 	1    9200 4600
 	1    0    0    -1
@@
 P 7950 4500
 F 0 "SW2" H 7950 4367 50  0000 C CNN
-F 1 "SW_SPST" H 7950 4276 50  0000 C CNN
+F 1 "SW_SPST" H 7950 4276 50  0001 C CNN
 F 2 "SensoriFeatherWing:SW_DS04-254-1L-01BK" H 7950 4500 50  0001 C CNN
 F 3 "~" H 7950 4500 50  0001 C CNN
+F 4 "2223-DS04-254-1L-01BK-ND" H 7950 4500 50  0001 C CNN "DKPN"
 	1    7950 4500
 	1    0    0    -1
@@
 	1    0    0    -1
 $EndComp
-Text Notes 7600 6050 0    50   ~ 0
-TODO:\n- Read datasheet of LDO -> caps? ESR?
+$Comp
+L Device:R R3
+U 1 1 5FB56AFD
+P 5350 4100
+F 0 "R3" V 5143 4100 50  0000 C CNN
+F 1 "120 Ω" V 5234 4100 50  0000 C CNN
+F 2 "Resistor_SMD:R_0805_2012Metric_Pad1.20x1.40mm_HandSolder" V 5280 4100 50  0001 C CNN
+F 3 "~" H 5350 4100 50  0001 C CNN
+	1    5350 4100
+	0    1    1    0
+$EndComp
+Wire Wire Line
+	5100 3750 5100 4100
+Wire Wire Line
+	5100 4100 5200 4100
+Connection ~ 5100 3750
+Wire Wire Line
+	5100 3750 5200 3750
+Wire Wire Line
+	5500 4100 5600 4100
+Wire Wire Line
+	5600 4100 5600 3750
+Connection ~ 5600 3750
+Wire Wire Line
+	5600 3750 5800 3750
 $EndSCHEMATC

Commit message: digikey part numbers
Parts:
- J5: DKPN (none) -> CP-002AH-ND
- J6: DKPN (none) -> 732-2745-ND
- R2: DKPN (none) -> 311-10KLDCT-ND
Changed lines of the file:
@@
 F 2 "TerminalBlock_4Ucon:TerminalBlock_4Ucon_1x02_P3.50mm_Horizontal" H 7550 2250 50  0001 C CNN
 F 3 "~" H 7550 2250 50  0001 C CNN
+F 4 "732-2745-ND" H 7550 2250 50  0001 C CNN "DKPN"
 	1    7550 2250
 	-1   0    0    1
@@
 F 2 "Connector_BarrelJack:BarrelJack_Horizontal" H 7500 1610 50  0001 C CNN
 F 3 "~" H 7500 1610 50  0001 C CNN
+F 4 "CP-002AH-ND" H 7450 1650 50  0001 C CNN "DKPN"
 	1    7450 1650
 	1    0    0    -1
@@
 F 2 "Resistor_SMD:R_0603_1608Metric_Pad0.98x0.95mm_HandSolder" H 8250 4800 50  0001 C CNN
 F 3 "~" H 8250 4800 50  0001 C CNN
+F 4 "311-10KLDCT-ND" H 8250 4800 50  0001 C CNN "DKPN"
 	1    8250 4800
 	1    0    0    -1
